File: kicad1.kicad_sch (KiCad schematic)
At the start: 44 parts

Commit message: An abomination of a first version
Connections:
- net -15V: now also C1.2, C10.1, C2.1, C3.2, C4.1, C5.2, C6.1, C7.2, C8.1, C9.2
Changed lines of the file:
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@@
 	(generator_version "9.0")
 	(paper "A4")
+	(rectangle
+		(start 175.26 59.69)
+		(end 283.21 138.43)
+		(stroke
+			(width 0)
+			(type default)
+			(color 19 255 4 1)
+		)
+		(fill
+			(type none)
+		)
+	)
+	(rectangle
+		(start 33.02 140.97)
+		(end 139.7 198.12)
+		(stroke
+			(width 0)
+			(type default)
+			(color 32 255 5 1)
+		)
+		(fill
+			(type none)
+		)
+	)
+	(rectangle
+		(start 64.77 57.15)
+		(end 172.72 119.38)
+		(stroke
+			(width 0)
+			(type default)
+			(color 19 255 4 1)
+		)
+		(fill
+			(type none)
+		)
+	)
+	(rectangle
+		(start 26.67 124.46)
+		(end 172.72 144.78)
+		(stroke
+			(width 0)
+			(type default)
+			(color 19 255 4 1)
+		)
+		(fill
+			(type none)
+		)
+	)
+	(rectangle
+		(start 17.78 13.97)
+		(end 88.9 59.69)
+		(stroke
+			(width 0)
+			(type default)
+			(color 14 255 17 1)
+		)
+		(fill
+			(type none)
+		)
+	)
 	(junction
 		(at 41.91 186.69)
@@
 	)
 	(junction
+		(at 88.9 167.64)
+		(diameter 0)
+		(color 0 0 0 0)
+	)
+	(junction
+		(at 49.53 167.64)
+		(diameter 0)
+		(color 0 0 0 0)
+	)
+	(junction
 		(at 120.65 97.155)
 		(diameter 0)
@@
 	)
 	(junction
+		(at 76.2 167.64)
+		(diameter 0)
+		(color 0 0 0 0)
+	)
+	(junction
 		(at 49.53 147.32)
 		(diameter 0)
@@
 	)
 	(junction
+		(at 63.5 167.64)
+		(diameter 0)
+		(color 0 0 0 0)
+	)
+	(junction
 		(at 63.5 147.32)
 		(diameter 0)
@@
 	)
 	(junction
+		(at 102.87 167.64)
+		(diameter 0)
+		(color 0 0 0 0)
+	)
+	(junction
 		(at 120.65 86.36)
 		(diameter 0)
@@
 	(wire
 		(pts
-			(xy 49.53 170.18) (xy 49.53 163.83)
+			(xy 49.53 170.18) (xy 49.53 167.64)
 		)
 		(stroke
@@
 	(wire
 		(pts
+			(xy 88.9 167.64) (xy 88.9 170.18)
+		)
+		(stroke
+			(width 0)
+			(type default)
+		)
+	)
+	(wire
+		(pts
 			(xy 124.46 121.92) (xy 120.65 121.92)
 		)
@@
 	(wire
 		(pts
+			(xy 76.2 167.64) (xy 76.2 163.83)
+		)
+		(stroke
+			(width 0)
+			(type default)
+		)
+	)
+	(wire
+		(pts
 			(xy 116.84 186.69) (xy 116.84 182.88)
 		)
@@
 	(wire
 		(pts
-			(xy 76.2 170.18) (xy 76.2 163.83)
+			(xy 76.2 170.18) (xy 76.2 167.64)
 		)
 		(stroke
@@
 	(wire
 		(pts
+			(xy 49.53 167.64) (xy 63.5 167.64)
+		)
+		(stroke
+			(width 0)
+			(type default)
+		)
+	)
+	(wire
+		(pts
 			(xy 90.17 82.55) (xy 90.17 66.04)
 		)
@@
 	(wire
 		(pts
+			(xy 102.87 167.64) (xy 133.35 167.64)
+		)
+		(stroke
+			(width 0)
+			(type default)
+		)
+	)
+	(wire
+		(pts
 			(xy 76.2 151.13) (xy 76.2 147.32)
 		)
@@
 	(wire
 		(pts
-			(xy 63.5 163.83) (xy 63.5 170.18)
+			(xy 63.5 163.83) (xy 63.5 167.64)
 		)
 		(stroke
@@
 	(wire
 		(pts
+			(xy 63.5 167.64) (xy 63.5 170.18)
+		)
+		(stroke
+			(width 0)
+			(type default)
+		)
+	)
+	(wire
+		(pts
 			(xy 69.85 60.96) (xy 96.52 60.96)
 		)
@@
 	(wire
 		(pts
+			(xy 63.5 167.64) (xy 76.2 167.64)
+		)
+		(stroke
+			(width 0)
+			(type default)
+		)
+	)
+	(wire
+		(pts
 			(xy 247.65 88.9) (xy 254 88.9)
 		)
@@
 	(wire
 		(pts
-			(xy 102.87 163.83) (xy 102.87 170.18)
+			(xy 102.87 163.83) (xy 102.87 167.64)
 		)
 		(stroke
@@
 	(wire
 		(pts
-			(xy 88.9 163.83) (xy 88.9 170.18)
+			(xy 88.9 163.83) (xy 88.9 167.64)
 		)
 		(stroke
@@
 	(wire
 		(pts
+			(xy 49.53 167.64) (xy 49.53 163.83)
+		)
+		(stroke
+			(width 0)
+			(type default)
+		)
+	)
+	(wire
+		(pts
+			(xy 102.87 167.64) (xy 102.87 170.18)
+		)
+		(stroke
+			(width 0)
+			(type default)
+		)
+	)
+	(wire
+		(pts
 			(xy 120.65 63.5) (xy 120.65 73.66)
 		)
@@
 	(wire
 		(pts
+			(xy 76.2 167.64) (xy 88.9 167.64)
+		)
+		(stroke
+			(width 0)
+			(type default)
+		)
+	)
+	(wire
+		(pts
 			(xy 120.65 97.155) (xy 120.65 97.79)
 		)
@@
 	(wire
 		(pts
-			(xy 41.91 167.64) (xy 133.35 167.64)
+			(xy 41.91 167.64) (xy 49.53 167.64)
 		)
 		(stroke
@@
 		)
 		(stroke
+			(width 0)
+			(type default)
+		)
+	)
+	(wire
+		(pts
+			(xy 88.9 167.64) (xy 102.87 167.64)
+		)
+		(stroke
