File: kicad1.kicad_pcb (KiCad board)
At the start: 2 copper layers, 100 x 80 mm, 44 parts

Commit message: An abomination of a first version
Parts:
- moved C10 282.9 mm to (105.0, 115.5), turned to -90 degrees
- moved C9 281.4 mm to (108.5, 103.0), turned to -90 degrees
- moved C8 278.1 mm to (108.5, 115.5), turned to -90 degrees
- moved C7 276.0 mm to (112.5, 103.0), turned to -90 degrees
- moved C6 273.0 mm to (112.5, 115.5), turned to -90 degrees
- moved R6 271.3 mm to (121.4, 89.9)
- moved uA741CP4 270.7 mm to (102.6, 84.8)
- moved C5 270.7 mm to (116.5, 103.0), turned to -90 degrees
- moved C4 268.0 mm to (116.5, 115.5), turned to -90 degrees
- moved R5 264.4 mm to (116.3, 80.3), turned to 90 degrees
- moved ROW_VERT/1X1 259.4 mm to (96.0, 84.9)
- moved TRIMMER/1K2 254.9 mm to (126.0, 72.1)
- moved C1 254.6 mm to (105.0, 103.0), turned to -90 degrees
- moved ROW_VERT/1X3 251.7 mm to (96.5, 109.5)
- moved C3 247.8 mm to (120.5, 103.0), turned to -90 degrees
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Connections:
- C1 pad 2: Net-(C1-Pad2) -> -15V
- C10 pad 1: Net-(C10-Pad1) -> -15V
- C2 pad 1: Net-(C1-Pad2) -> -15V
- C3 pad 2: Net-(C3-Pad2) -> -15V
- C4 pad 1: Net-(C3-Pad2) -> -15V
- C5 pad 2: Net-(C5-Pad2) -> -15V
- C6 pad 1: Net-(C5-Pad2) -> -15V
- C7 pad 2: Net-(C7-Pad2) -> -15V
- C8 pad 1: Net-(C7-Pad2) -> -15V
- C9 pad 2: Net-(C10-Pad1) -> -15V
Routing:
- net -15V: track 0.00 -> 304.9 mm
- net +15V: track 0.00 -> 269.6 mm
- net Net-(R15-Pad1): track 0.00 -> 105.2 mm
- net Net-(uA741CP2--): track 0.00 -> 49.8 mm
- net Net-(BC547_1-E): track 0.00 -> 43.9 mm
- net Net-(uA741CP3--): track 0.00 -> 33.9 mm
- net Net-(C17-Pad2): track 0.00 -> 24.6 mm
- net Net-(BC547_1-B): track 0.00 -> 20.2 mm
- net Net-(uA741CP1--): track 0.00 -> 19.8 mm
- net Net-(uA741CP2-+): track 0.00 -> 19.8 mm
- net Net-(uA741CP4--): track 0.00 -> 18.8 mm
- net Net-(R11-Pad2): track 0.00 -> 16.3 mm
- net Net-(R10-Pad1): track 0.00 -> 14.8 mm
- net Net-(R5-Pad1): track 0.00 -> 10.9 mm
- net Net-(R3-Pad1): track 0.00 -> 8.00 mm
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
Commit message: epätoivoinen versio ennen resettiä
Parts:
- moved R18 2.67 mm to (180.9, 75.6)
- moved R11 2.31 mm to (146.5, 48.5)
- moved R2 1.53 mm to (103.4, 51.4)
- moved R1 0.93 mm to (99.3, 51.4), turned to 90 degrees
- moved ROW_VERT/1X1 0.36 mm to (96.4, 84.9)
Connections:
- C1 pad 2: -15V -> GND
- C10 pad 1: -15V -> GND
- C13 pad 2: unconnected-(C13-Pad2) -> GND
- C14 pad 1: unconnected-(C14-Pad1) -> GND
- C15 pad 1: -15V -> GND
- C16 pad 1: -15V -> GND
- C2 pad 1: -15V -> GND
- C3 pad 2: -15V -> GND
- C4 pad 1: -15V -> GND
- C5 pad 2: -15V -> GND
- C6 pad 1: -15V -> GND
- C7 pad 2: -15V -> GND
- C8 pad 1: -15V -> GND
- C9 pad 2: -15V -> GND
- R1 pad 1: +15V -> Net-(ROW_VERT/1X1-Pin_1)
- R10 pad 2: +15V -> Net-(uA741CP1-+)
- R17 pad 1: -15V -> GND
- R2 pad 1: +15V -> Net-(ROW_VERT/1X1-Pin_1)
- R3 pad 1: Net-(R3-Pad1) -> Net-(uA741CP1-+)
- R4 pad 1: Net-(R3-Pad1) -> Net-(uA741CP1-+)
- R7 pad 2: -15V -> GND
- ROW_VERT/1X1 pad 1: +15V -> Net-(ROW_VERT/1X1-Pin_1)
- ROW_VERT/1X1 pad 2: -15V -> Net-(ROW_VERT/1X1-Pin_2)
- ROW_VERT/1X1 pad 3: -15V -> GND
- ROW_VERT/1X2 pad 2: -15V -> GND
- ROW_VERT/1X3 pad 2: -15V -> GND
- TRIMMER/1K1 pad 2: -15V -> GND
- uA741CP1 pad 3: +15V -> Net-(uA741CP1-+)
- uA741CP1 pad 4: unconnected-(uA741CP1-V--Pad4) -> -15V
- uA741CP1 pad 7: unconnected-(uA741CP1-V+-Pad7) -> +15V
- uA741CP2 pad 4: unconnected-(uA741CP2-V--Pad4) -> -15V
- uA741CP2 pad 7: unconnected-(uA741CP2-V+-Pad7) -> +15V
- uA741CP3 pad 4: unconnected-(uA741CP3-V--Pad4) -> -15V
- uA741CP3 pad 7: unconnected-(uA741CP3-V+-Pad7) -> +15V
- uA741CP4 pad 3: -15V -> Net-(ROW_VERT/1X1-Pin_2)
- uA741CP4 pad 4: unconnected-(uA741CP4-V--Pad4) -> -15V
- uA741CP4 pad 7: unconnected-(uA741CP4-V+-Pad7) -> +15V
Routing:
- net GND: track 0.00 -> 277.1 mm
- net -15V: track 304.9 -> 95.8 mm
- net Net-(R15-Pad1): track 105.2 -> 11.8 mm
- net Net-(ROW_VERT/1X1-Pin_1): track 0.00 -> 52.5 mm
- net Net-(uA741CP1-+): track 0.00 -> 50.5 mm
- net Net-(BC547_1-E): track 43.9 -> 5.70 mm
- net +15V: track 269.6 -> 299.7 mm
- net Net-(uA741CP2-+): track 19.8 -> 6.24 mm
- net Net-(uA741CP4--): track 18.8 -> 28.5 mm
- net Net-(R3-Pad1): track 8.00 -> 0.00 mm
- net Net-(ROW_VERT/1X1-Pin_2): track 0.00 -> 7.29 mm
- net Net-(uA741CP2--): track 49.8 -> 47.1 mm
- net Net-(uA741CP1--): track 19.8 -> 17.2 mm
- net Net-(R11-Pad2): track 16.3 -> 13.9 mm

Commit message: done
Parts:
- moved uA741CP3 58.1 mm to (132.3, 93.4), turned to 0 degrees
- moved C2 50.7 mm to (165.4, 91.9), turned to 90 degrees
- moved C3 50.6 mm to (160.2, 71.6), turned to 90 degrees
- moved C13 50.1 mm to (123.5, 55.1), turned to 0 degrees
- moved R7 47.0 mm to (97.9, 117.2), turned to 90 degrees
- moved R9 45.3 mm to (139.9, 71.9), turned to 180 degrees
- moved uA741CP1 42.4 mm to (109.9, 79.1), turned to 180 degrees
- moved ROW_VERT/1X3 41.4 mm to (137.3, 116.6), turned to 180 degrees
- moved R8 41.2 mm to (126.6, 72.1)
- moved R11 40.2 mm to (118.1, 77.0), turned to 90 degrees
- moved C6 39.4 mm to (90.1, 83.1), turned to 0 degrees
- moved C7 39.3 mm to (95.1, 67.8), turned to 180 degrees
- moved C14 37.4 mm to (157.5, 92.4), turned to 90 degrees
- moved C9 35.7 mm to (143.5, 96.0), turned to 0 degrees
- moved R6 33.5 mm to (102.0, 117.2), turned to -90 degrees
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Connections:
- R16 pad 1: +15V -> Net-(ROW_VERT/1X2-Pin_1)
- R21 pad 1: +15V -> Net-(ROW_VERT/1X2-Pin_1)
- ROW_VERT/1X2 pad 1: +15V -> Net-(ROW_VERT/1X2-Pin_1)
Routing:
- net GND: track 277.1 -> 402.3 mm
- net -15V: track 95.8 -> 166.1 mm
- net Net-(uA741CP2-+): track 6.24 -> 39.2 mm
- net Net-(uA741CP1-+): track 50.5 -> 20.8 mm
- net Net-(R11-Pad2): track 13.9 -> 41.5 mm
- net +15V: track 299.7 -> 326.6 mm
- net Net-(R15-Pad1): track 11.8 -> 29.9 mm
- net Net-(BC547_1-B): track 20.2 -> 2.90 mm
- net Net-(uA741CP4--): track 28.5 -> 13.0 mm
- net Net-(ROW_VERT/1X1-Pin_2): track 7.29 -> 20.6 mm
- net Net-(ROW_VERT/1X2-Pin_1): track 0.00 -> 12.9 mm
- net Net-(R10-Pad1): track 14.8 -> 4.31 mm
- net Net-(BC547_1-E): track 5.70 -> 13.1 mm
- net Net-(C17-Pad2): track 24.6 -> 19.2 mm
- net Net-(uA741CP3--): track 33.9 -> 28.7 mm
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- added copper zone on B.Cu, net +15V
